File: Project_02/EAGLE/Actual/Etch-a-sketch.brd (EAGLE design)
At the start: 62.5 x 81.3 mm, 24 parts, among them J1 292303-1, J2 SPI_LCD, SW1 PUSH_BUTTON, SW2 PUSH_BUTTON, U1 POCKETBEAGLE

Commit message: etch the sketch
Parts:
- moved R2 199.9 mm to (100.3, 41.9)
- moved SW2 199.9 mm to (106.0, 52.7)
- moved D3 173.9 mm to (80.0, 62.9)
- moved R6 173.9 mm to (84.5, 46.4)
- moved J2 92.0 mm to (43.2, 27.3)
- moved R4 59.7 mm to (-14.0, 54.6)
- moved SW1 59.7 mm to (-22.9, 54.6)
- moved R1 57.6 mm to (-1.27, 45.7)
Routing:
- net LEFT_BUTTON: track 21.1 -> 81.7 mm
- net BUZZER: track 25.0 -> 73.8 mm
- net LEFT_POTENTIOMETER: track 49.6 -> 95.0 mm
- net AGND: track 45.2 -> 66.7 mm
- net VDD_1P8V: track 39.4 -> 53.2 mm
